File: Eagle/DigitMux.brd (EAGLE design)
At the start: 100 x 100 mm, 205 parts, among them CN2 1X04_SMD_STRAIGHT_COMBO, J1 RA 6Pin SMD

Commit message: Silk cleanup
Parts:
- moved J1A 1.59 mm to (15.2, 97.8)
- moved J1B 1.59 mm to (40.6, 97.8)
- moved J1C 1.59 mm to (66.0, 97.8)
- moved CN1 1.27 mm to (50.8, 2.54)
- moved J1 1.27 mm to (71.1, 2.54)
- moved CN2 1.26 mm to (58.4, 2.54)
Routing:
- net N$2: track 4.71 -> 3.12 mm
- net N$13: track 4.71 -> 3.12 mm
- net N$21: track 4.71 -> 3.12 mm
- net N$95: track 15.3 -> 14.1 mm
- net N$88: track 19.1 -> 20.4 mm
- net N$96: track 19.8 -> 18.5 mm
- net N$94: track 11.6 -> 10.4 mm
- net N$92: track 14.7 -> 16.0 mm
- net GND: track 329.7 -> 328.5 mm
- net N$22: track 4.07 -> 2.86 mm
- net N$6: track 4.07 -> 2.86 mm
- net N$14: track 4.07 -> 2.86 mm
- net N$60: track 189.5 -> 188.6 mm
- net N$25: track 2.99 -> 3.83 mm
- net N$17: track 2.99 -> 3.65 mm
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Other:
- board text removed: "15"
- board text removed: "23"
- board text removed: "7"
